Commit message: feat(assembler): 파트 결합 인터랙티브 조립 GUI + mounts.yaml 연동
rda_robot_assembler: PyQt5 + pyvista 내장 3D 조립 도구
- part_registry: 5슬롯(base/arm/endeffector/sensor1/sensor2)·모델 레지스트리
- urdf_loader: xacro→urdf, yourdfpy 로드, package:// 리졸버, 프레임 FK/anchor
- assembly: topological 배치(parent_frame_world @ mount @ inv(anchor))
- app: 좌 슬롯 / 중앙 3D뷰(부착프레임 축) / 우 결합설정(부모TF·XYZ·RPY 라이브)
  · mounts.yaml 저장/불러오기/초기화

rda_robot_description:
- config/mounts.yaml: 결합값(parent_frame·xyz·rpy·센서모델)
- rda_robot.urdf.xacro: mounts.yaml 을 읽어 통합(센서 d405/d435i 조건부),
  mounts_file:= 인자 override 지원

검증: 로더/배치 헤드리스 OK, 앱 실행·렌더 안정, yaml override→xacro 반영,
colcon 빌드 + ros2 run rda_robot_assembler assembler

Co-Authored-By: Claude Opus 4.8 (1M context) <noreply@anthropic.com>

File: rda_robot_description/urdf/rda_robot.urdf.xacro (robot description, xacro)
@@ -1,47 +1,54 @@
 <?xml version="1.0"?>
 <!--
-  rda_robot — 4개 파트 통합 URDF 초안 (2주차 산출물)
-  구성: ⓐScout 2.0(모바일, 루트) + ⓑRB5-850e(팔) + ⓒOnRobot RG2(그리퍼)
-        + ⓓD405(eye-in-hand) + D435i(eye-to-hand)
-  주의:
-    - mount origin(장착 위치/자세)은 도면 확정 전 초안 추정값 = TODO.
-    - RB5는 rb_6dof 매크로 prefix 버그로 무접두(link0..6,tcp) 사용. 상세: docs/파트규약-비교.md
-  검증: xacro→urdf, check_urdf 단일 트리, RViz2 표시.
+  rda_robot — 4개 파트 통합 URDF (mounts.yaml 기반)
+  구성: ⓐScout 2.0(루트) + ⓑRB5-850e(팔) + ⓒOnRobot RG2(그리퍼)
+        + ⓓ센서1(eye-in-hand) + 센서2(eye-to-hand)
+  결합값(parent_frame·xyz·rpy)은 config/mounts.yaml 에서 읽는다.
+  → rda_robot_assembler 앱으로 mounts.yaml 을 편집하면 여기 통합 형상이 바뀐다.
+  주의: RB5 는 rb_6dof prefix 버그로 무접두(link0..6). 상세: docs/파트규약-비교.md
 -->
 <robot xmlns:xacro="http://www.ros.org/wiki/xacro" name="rda_robot">
-  <!-- ============ ⓐ 모바일: Scout 2.0 (매크로 아님 → base_link 루트 직접 정의) ============ -->
+  <xacro:arg name="mounts_file" default="$(find rda_robot_description)/config/mounts.yaml"/>
+  <xacro:property name="M" value="${xacro.load_yaml('$(arg mounts_file)')['mounts']}"/>
+  <!-- ============ ⓐ 모바일: Scout 2.0 (루트 base_link) ============ -->
   <xacro:include filename="$(find scout_description)/urdf/scout_v2.xacro"/>
   <!-- ============ ⓑ 로봇팔: RB5-850e ============ -->
   <xacro:include filename="$(find rbpodo_description)/robots/rb_6dof.xacro"/>
-  <!-- TODO: 실제 팔 장착 위치(스카웃 상판 높이/오프셋) 확정 필요 -->
+  <xacro:property name="am" value="${M['arm']}"/>
   <joint name="arm_mount_joint" type="fixed">
-    <parent link="base_link"/>
+    <parent link="${am['parent_frame']}"/>
     <child link="link0"/>
-    <origin xyz="0.0 0.0 0.25" rpy="0 0 0"/>
+    <origin xyz="${am['xyz'][0]} ${am['xyz'][1]} ${am['xyz'][2]}"
+            rpy="${am['rpy'][0]} ${am['rpy'][1]} ${am['rpy'][2]}"/>
   </joint>
   <xacro:rb_6dof model_id="rb5_850e" prefix="" tcp_name="tcp"/>
-  <!-- ============ ⓒ 엔드이펙터: OnRobot RG2 (팔 tcp 에 부착) ============ -->
+  <!-- ============ ⓒ 엔드이펙터: OnRobot RG2 ============ -->
   <xacro:include filename="$(find rda_robot_description)/urdf/parts/endeffector/onrobot_rg2_macro.xacro"/>
-  <!-- TODO: 실제 플랜지-그리퍼 어댑터 오프셋 확정 필요 -->
-  <xacro:onrobot_rg2 parent="tcp" prefix="">
-    <origin xyz="0 0 0" rpy="0 0 0"/>
+  <xacro:property name="em" value="${M['endeffector']}"/>
+  <xacro:onrobot_rg2 parent="${em['parent_frame']}" prefix="">
+    <origin xyz="${em['xyz'][0]} ${em['xyz'][1]} ${em['xyz'][2]}"
+            rpy="${em['rpy'][0]} ${em['rpy'][1]} ${em['rpy'][2]}"/>
   </xacro:onrobot_rg2>
-  <!-- ============ ⓓ 센서 1: D405 (eye-in-hand, 그리퍼 손목에 부착) ============ -->
+  <!-- ============ ⓓ 센서: RealSense (모델별 매크로 선택) ============ -->
   <xacro:include filename="$(find realsense2_description)/urdf/_d405.urdf.xacro"/>
-  <!-- TODO: 실제 eye-in-hand 브래킷 위치 확정 필요 -->
-  <xacro:sensor_d405 parent="rg2_hand" name="d405" use_nominal_extrinsics="true">
-    <origin xyz="0.02 0.0 0.03" rpy="0 0 0"/>
-  </xacro:sensor_d405>
-  <!-- ============ ⓓ 센서 2: D435i (eye-to-hand, 베이스 마스트에 부착) ============ -->
   <xacro:include filename="$(find realsense2_description)/urdf/_d435i.urdf.xacro"/>
-  <!-- 초안 마스트: 베이스 위 고정 프레임 (TODO: 실제 마스트 형상/높이) -->
-  <link name="sensor_mast"/>
-  <joint name="mast_joint" type="fixed">
-    <parent link="base_link"/>
-    <child link="sensor_mast"/>
-    <origin xyz="-0.25 0.0 0.6" rpy="0 0.3 0"/>
-  </joint>
-  <xacro:sensor_d435i parent="sensor_mast" name="d435i" use_nominal_extrinsics="true">
-    <origin xyz="0 0 0" rpy="0 0 0"/>
-  </xacro:sensor_d435i>
+  <!-- 센서 부착 매크로: 모델에 따라 d405/d435i 인스턴스화 -->
+  <xacro:macro name="mount_sensor" params="key">
+    <xacro:property name="s" value="${M[key]}"/>
+    <xacro:property name="sname" value="${s['model']}"/>
+    <xacro:if value="${sname == 'd405'}">
+      <xacro:sensor_d405 parent="${s['parent_frame']}" name="${sname}" use_nominal_extrinsics="true">
+        <origin xyz="${s['xyz'][0]} ${s['xyz'][1]} ${s['xyz'][2]}"
+                rpy="${s['rpy'][0]} ${s['rpy'][1]} ${s['rpy'][2]}"/>
+      </xacro:sensor_d405>
+    </xacro:if>
+    <xacro:if value="${sname == 'd435i'}">
+      <xacro:sensor_d435i parent="${s['parent_frame']}" name="${sname}" use_nominal_extrinsics="true">
+        <origin xyz="${s['xyz'][0]} ${s['xyz'][1]} ${s['xyz'][2]}"
+                rpy="${s['rpy'][0]} ${s['rpy'][1]} ${s['rpy'][2]}"/>
+      </xacro:sensor_d435i>
+    </xacro:if>
+  </xacro:macro>
+  <xacro:mount_sensor key="sensor1"/>
+  <xacro:mount_sensor key="sensor2"/>
 </robot>

Commit message: feat(description): 통합 URDF 모델 자동 스위칭 (mounts.yaml 기반)
base/arm/endeffector 도 센서처럼 mounts.yaml 로 스위칭:
- 베이스: models.base 값으로 xacro:if 조건부 include(루트 링크 정의).
- 팔/그리퍼: mounts.<slot>.model 값으로 조건부 매크로 인스턴스화
  (include+mount joint+매크로 호출을 슬롯당 분기 블록으로).
- 조립기 드롭다운에서 모델 바꿔 저장 → 통합 형상 자동 반영.
- Humble xacro 조건부 include 동작 확인. 새 모델은 분기 블록 복사로 추가
  (모델마다 매크로 인터페이스·루트링크 달라 슬롯당 블록 필요 — 주석 안내).
- 검증: 기본 mounts→42링크 단일트리(기존 동일), 미등록 id→해당 슬롯 제외,
  센서 d405→d435i 스왑 반영. 전체 launch(rsp+monitor) 정상.

Co-Authored-By: Claude Opus 4.8 (1M context) <noreply@anthropic.com>

File: rda_robot_description/urdf/rda_robot.urdf.xacro (robot description, xacro)
@@ -1,37 +1,59 @@
 <?xml version="1.0"?>
 <!--
-  rda_robot — 4개 파트 통합 URDF (mounts.yaml 기반)
-  구성: ⓐScout 2.0(루트) + ⓑRB5-850e(팔) + ⓒOnRobot RG2(그리퍼)
-        + ⓓ센서1(eye-in-hand) + 센서2(eye-to-hand)
-  결합값(parent_frame·xyz·rpy)은 config/mounts.yaml 에서 읽는다.
-  → rda_robot_assembler 앱으로 mounts.yaml 을 편집하면 여기 통합 형상이 바뀐다.
+  rda_robot — 4개 파트 통합 URDF (mounts.yaml 기반, 모델 자동 스위칭)
+  구성: ⓐ베이스(모바일) + ⓑ로봇팔 + ⓒ엔드이펙터(그리퍼) + ⓓ센서1·2
+  ■ 모델/결합값 출처: config/mounts.yaml (rda_robot_assembler 앱이 저장)
+    - models.base           : 베이스 모델 id
+    - mounts.<slot>.model    : 팔/그리퍼/센서 모델 id
+    - mounts.<slot>.parent_frame / xyz / rpy : 결합 위치
+    → 앱 드롭다운에서 모델을 바꿔 저장하면 여기 통합 형상이 자동으로 바뀐다.
+  ■ 새 모델 추가법: 해당 슬롯의 <xacro:if value="${...=='새id'}"> 블록을 복사해
+    include(있으면)·mount joint·매크로 호출을 그 모델에 맞게 채운다.
+    (각 모델은 매크로 인터페이스·루트 링크명이 달라 슬롯당 분기 블록이 필요하다.)
   주의: RB5 는 rb_6dof prefix 버그로 무접두(link0..6). 상세: docs/파트규약-비교.md
 -->
 <robot xmlns:xacro="http://www.ros.org/wiki/xacro" name="rda_robot">
   <xacro:arg name="mounts_file" default="$(find rda_robot_description)/config/mounts.yaml"/>
-  <xacro:property name="M" value="${xacro.load_yaml('$(arg mounts_file)')['mounts']}"/>
-  <!-- ============ ⓐ 모바일: Scout 2.0 (루트 base_link) ============ -->
-  <xacro:include filename="$(find scout_description)/urdf/scout_v2.xacro"/>
-  <!-- ============ ⓑ 로봇팔: RB5-850e ============ -->
-  <xacro:include filename="$(find rbpodo_description)/robots/rb_6dof.xacro"/>
+  <xacro:property name="Y" value="${xacro.load_yaml('$(arg mounts_file)')}"/>
+  <xacro:property name="M" value="${Y['mounts']}"/>
+  <xacro:property name="SEL" value="${Y['models']}"/>
+  <!-- ============ ⓐ 베이스(모바일) — models.base 로 스위칭 ============ -->
+  <xacro:property name="bname" value="${SEL['base']}"/>
+  <xacro:if value="${bname == 'scout_v2'}">
+    <xacro:include filename="$(find scout_description)/urdf/scout_v2.xacro"/>
+  </xacro:if>
+  <!-- 새 베이스 추가:
+  <xacro:if value="${bname == '새베이스id'}">
+    <xacro:include filename="$(find 새패키지)/urdf/새베이스.xacro"/>
+  </xacro:if>
+  -->
+  <!-- ============ ⓑ 로봇팔 — mounts.arm.model 로 스위칭 ============ -->
   <xacro:property name="am" value="${M['arm']}"/>
-  <joint name="arm_mount_joint" type="fixed">
-    <parent link="${am['parent_frame']}"/>
-    <child link="link0"/>
-    <origin xyz="${am['xyz'][0]} ${am['xyz'][1]} ${am['xyz'][2]}"
-            rpy="${am['rpy'][0]} ${am['rpy'][1]} ${am['rpy'][2]}"/>
-  </joint>
-  <xacro:rb_6dof model_id="rb5_850e" prefix="" tcp_name="tcp"/>
-  <!-- ============ ⓒ 엔드이펙터: OnRobot RG2 ============ -->
-  <xacro:include filename="$(find rda_robot_description)/urdf/parts/endeffector/onrobot_rg2_macro.xacro"/>
+  <xacro:property name="aname" value="${am['model']}"/>
+  <xacro:if value="${aname == 'rb5_850e'}">
+    <xacro:include filename="$(find rbpodo_description)/robots/rb_6dof.xacro"/>
+    <joint name="arm_mount_joint" type="fixed">
+      <parent link="${am['parent_frame']}"/>
+      <child link="link0"/>
+      <origin xyz="${am['xyz'][0]} ${am['xyz'][1]} ${am['xyz'][2]}"
+              rpy="${am['rpy'][0]} ${am['rpy'][1]} ${am['rpy'][2]}"/>
+    </joint>
+    <xacro:rb_6dof model_id="rb5_850e" prefix="" tcp_name="tcp"/>
+  </xacro:if>
+  <!-- 새 팔 추가: include + arm_mount_joint(child=그 팔의 루트링크) + 그 팔 매크로 호출 -->
+  <!-- ============ ⓒ 엔드이펙터 — mounts.endeffector.model 로 스위칭 ============ -->
   <xacro:property name="em" value="${M['endeffector']}"/>
-  <xacro:onrobot_rg2 parent="${em['parent_frame']}" prefix="">
-    <origin xyz="${em['xyz'][0]} ${em['xyz'][1]} ${em['xyz'][2]}"
-            rpy="${em['rpy'][0]} ${em['rpy'][1]} ${em['rpy'][2]}"/>
-  </xacro:onrobot_rg2>
-  <!-- ============ ⓓ 센서: RealSense (모델별 매크로 선택) ============ -->
+  <xacro:property name="ename" value="${em['model']}"/>
+  <xacro:if value="${ename == 'onrobot_rg2'}">
+    <xacro:include filename="$(find rda_robot_description)/urdf/parts/endeffector/onrobot_rg2_macro.xacro"/>
+    <xacro:onrobot_rg2 parent="${em['parent_frame']}" prefix="">
+      <origin xyz="${em['xyz'][0]} ${em['xyz'][1]} ${em['xyz'][2]}"
+              rpy="${em['rpy'][0]} ${em['rpy'][1]} ${em['rpy'][2]}"/>
+    </xacro:onrobot_rg2>
+  </xacro:if>
+  <!-- 새 그리퍼 추가: include + 그 그리퍼 매크로 호출(parent=${em['parent_frame']}) -->
+  <!-- ============ ⓓ 센서: RealSense (mounts.sensorN.model 로 스위칭) ============ -->
   <xacro:include filename="$(find realsense2_description)/urdf/_d405.urdf.xacro"/>
   <xacro:include filename="$(find realsense2_description)/urdf/_d435i.urdf.xacro"/>
-  <!-- 센서 부착 매크로: 모델에 따라 d405/d435i 인스턴스화 -->
   <xacro:macro name="mount_sensor" params="key">
     <xacro:property name="s" value="${M[key]}"/>

Commit message: fix(description): 분기 없는 모델 선택 시 조용한 슬롯 누락 → 즉시 실패
mounts.yaml 이 xacro:if 분기가 없는 모델(28종 중 21종)을 가리키면 xacro 가
exit=0 으로 통과하면서 해당 슬롯을 통째로 누락시켰다. 하위 마운트가 붕 떠
check_urdf/rsp 에서야 "parent link [tcp] not found" 로 터져 원인 추적이 어려웠다
(42→34링크, display·moveit launch 둘 다 기동 불가).

슬롯별 SUPPORTED_* 목록 + xacro:check_slot 매크로로 xacro.fatal() 즉시 실패시킨다.
메시지에 슬롯명·고른 모델·지원 목록·조치법을 담아 launch 출력까지 그대로 노출된다.

폴백(기본모델 자동 대체)은 의도적으로 채택하지 않음: 고르지도 않은 형상 위에서
도달권·SRDF·경로계획이 계산되는 게 기동 실패보다 위험하다. 근본 해결은
Python URDF 컴포저이며, 이 방어는 그때까지의 안전망이다.

검증:
- arm__rb10_1300e(현 mounts.yaml): exit=2 + 명확한 메시지, launch 에도 노출
- base/endeffector/sensor2 슬롯 각각 오탐 없이 발동(슬롯 키 정확히 표기)
- rb5_850e(지원 모델): 42링크 + check_urdf 통과 = 회귀 없음

Co-Authored-By: Claude Opus 4.8 (1M context) <noreply@anthropic.com>

File: rda_robot_description/urdf/rda_robot.urdf.xacro (robot description, xacro)
@@ -11,4 +11,11 @@
     include(있으면)·mount joint·매크로 호출을 그 모델에 맞게 채운다.
     (각 모델은 매크로 인터페이스·루트 링크명이 달라 슬롯당 분기 블록이 필요하다.)
+    ★ 분기를 추가했으면 아래 SUPPORTED_* 목록에도 그 id 를 반드시 넣을 것.
+  ■ 지원 모델 한계(2026-07-16): 조립기 드롭다운에는 28종이 뜨지만, 통합 URDF 는 아래
+    SUPPORTED_* 에 있는 7종만 반영한다. 지원 밖 모델을 고르면 xacro 가 조용히 슬롯을
+    누락시켜 엉뚱한 곳(check_urdf/rsp)에서 터졌었다 → xacro.check_slot 으로 즉시 실패시킨다.
+    폴백(기본모델로 조용히 대체)은 의도적으로 넣지 않는다: 고르지도 않은 형상 위에서
+    도달권·SRDF·경로계획이 계산되는 게 기동 실패보다 위험하다.
+    근본 해결은 Python URDF 컴포저(작업중) — 완료되면 이 한계와 방어는 사라진다.
   주의: RB5 는 rb_6dof prefix 버그로 무접두(link0..6). 상세: docs/파트규약-비교.md
 -->
@@ -18,6 +25,24 @@
   <xacro:property name="M" value="${Y['mounts']}"/>
   <xacro:property name="SEL" value="${Y['models']}"/>
+  <!-- ============ 슬롯 모델 방어 — 분기 없는 모델이면 즉시 실패 ============ -->
+  <xacro:property name="SUPPORTED_BASE" value="${['scout_v2']}"/>
+  <xacro:property name="SUPPORTED_ARM" value="${['rb5_850e']}"/>
+  <xacro:property name="SUPPORTED_EE" value="${['onrobot_rg2']}"/>
+  <xacro:property name="SUPPORTED_SENSOR" value="${['d405', 'd435i']}"/>
+  <xacro:macro name="check_slot" params="slot name supported">
+    <xacro:if value="${name not in supported}">
+      ${xacro.fatal(
+        slot + " 슬롯: 모델 '" + str(name) + "' 는 통합 URDF 에 반영할 수 없습니다"
+        + " (해당 xacro:if 분기 없음)."
+        + "  ■ 이 슬롯이 지원하는 모델: " + ', '.join(supported)
+        + "  ■ 조치: config/mounts.yaml 에서 위 모델 중 하나로 바꾸거나,"
+        + " Python URDF 컴포저(작업중) 완료 후 재시도하세요."
+        + "  ※ 조립기 드롭다운의 28종이 곧 통합 URDF 지원 목록은 아닙니다."
+      )}
+    </xacro:if>
+  </xacro:macro>
   <!-- ============ ⓐ 베이스(모바일) — models.base 로 스위칭 ============ -->
   <xacro:property name="bname" value="${SEL['base']}"/>
+  <xacro:check_slot slot="base" name="${bname}" supported="${SUPPORTED_BASE}"/>
   <xacro:if value="${bname == 'scout_v2'}">
     <xacro:include filename="$(find scout_description)/urdf/scout_v2.xacro"/>
@@ -31,4 +56,5 @@
   <xacro:property name="am" value="${M['arm']}"/>
   <xacro:property name="aname" value="${am['model']}"/>
+  <xacro:check_slot slot="arm" name="${aname}" supported="${SUPPORTED_ARM}"/>
   <xacro:if value="${aname == 'rb5_850e'}">
     <xacro:include filename="$(find rbpodo_description)/robots/rb_6dof.xacro"/>
@@ -45,4 +71,5 @@
   <xacro:property name="em" value="${M['endeffector']}"/>
   <xacro:property name="ename" value="${em['model']}"/>
+  <xacro:check_slot slot="endeffector" name="${ename}" supported="${SUPPORTED_EE}"/>
   <xacro:if value="${ename == 'onrobot_rg2'}">
     <xacro:include filename="$(find rda_robot_description)/urdf/parts/endeffector/onrobot_rg2_macro.xacro"/>
@@ -59,4 +86,5 @@
     <xacro:property name="s" value="${M[key]}"/>
     <xacro:property name="sname" value="${s['model']}"/>
+    <xacro:check_slot slot="${key}" name="${sname}" supported="${SUPPORTED_SENSOR}"/>
     <xacro:if value="${sname == 'd405'}">
       <xacro:sensor_d405 parent="${s['parent_frame']}" name="${sname}" use_nominal_extrinsics="true">
